File: Boards/Coax2wireinterface/wire2coax.brd (EAGLE design)
At the start: 647.7 x 87.6 mm, 0 parts

Commit message: Added Coax2Wire interface board, updated the README.md file with the coax datasheet and a posible replacement for pico BNC connectors
Routing:
- added copper zone on layer 16, net GROUND
- added copper zone on layer 1, net S$1
Other:
- board size 647.7 x 87.6 mm -> 12 x 12 mm
Changed lines of the file:
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@@
 <drawing>
 <settings>
-<setting alwaysvectorfont="no"/>
+<setting alwaysvectorfont="yes"/>
 <setting verticaltext="up"/>
 </settings>
-<grid distance="5" unitdist="mil" unit="mm" style="lines" multiple="1" display="yes" altdistance="0.003125" altunitdist="mic" altunit="mm"/>
+<grid distance="1" unitdist="mm" unit="mm" style="lines" multiple="1" display="yes" altdistance="0.1" altunitdist="mm" altunit="mm"/>
 <layers>
 <layer number="1" name="Top" color="4" fill="1" visible="yes" active="yes"/>
@@
 <layer number="27" name="tValues" color="7" fill="1" visible="yes" active="yes"/>
 <layer number="28" name="bValues" color="7" fill="1" visible="yes" active="yes"/>
-<layer number="29" name="tStop" color="7" fill="3" visible="no" active="yes"/>
-<layer number="30" name="bStop" color="7" fill="6" visible="no" active="yes"/>
+<layer number="29" name="tStop" color="7" fill="3" visible="yes" active="yes"/>
+<layer number="30" name="bStop" color="7" fill="6" visible="yes" active="yes"/>
 <layer number="31" name="tCream" color="7" fill="4" visible="no" active="yes"/>
 <layer number="32" name="bCream" color="7" fill="5" visible="no" active="yes"/>
 <layer number="33" name="tFinish" color="6" fill="3" visible="no" active="yes"/>
-<layer number="34" name="bFinish" color="6" fill="6" visible="no" active="yes"/>
+<layer number="34" name="bFinish" color="6" fill="6" visible="yes" active="yes"/>
 <layer number="35" name="tGlue" color="7" fill="4" visible="no" active="yes"/>
 <layer number="36" name="bGlue" color="7" fill="5" visible="no" active="yes"/>
@@
 <layer number="45" name="Holes" color="7" fill="1" visible="yes" active="yes"/>
 <layer number="46" name="Milling" color="3" fill="1" visible="no" active="yes"/>
-<layer number="47" name="Measures" color="7" fill="1" visible="yes" active="yes"/>
+<layer number="47" name="Measures" color="7" fill="1" visible="no" active="yes"/>
 <layer number="48" name="Document" color="7" fill="1" visible="yes" active="yes"/>
 <layer number="49" name="Reference" color="7" fill="1" visible="yes" active="yes"/>
@@
 <board>
 <plain>
-<wire x1="647.7" y1="-7.62" x2="643.89" y2="-11.43" width="0.1524" layer="20" curve="-90"/>
-<wire x1="3.937" y1="0" x2="70.104" y2="0" width="0.1524" layer="20"/>
-<wire x1="73.787" y1="3.683" x2="73.787" y2="72.263" width="0.1524" layer="20"/>
-<wire x1="69.85" y1="76.2" x2="3.937" y2="76.2" width="0.1524" layer="20"/>
-<wire x1="0" y1="72.263" x2="0" y2="3.937" width="0.1524" layer="20"/>
-<wire x1="0" y1="72.263" x2="3.937" y2="76.2" width="0.1524" layer="20" curve="-90"/>
-<wire x1="3.937" y1="0" x2="0" y2="3.937" width="0.1524" layer="20" curve="-90"/>
-<wire x1="70.104" y1="0" x2="73.787" y2="3.683" width="0.1524" layer="20" curve="90"/>
-<wire x1="73.787" y1="72.263" x2="69.85" y2="76.2" width="0.1524" layer="20" curve="90"/>
-<circle x="7.897" y="7.632" radius="1.1305" width="0.1524" layer="20"/>
-<circle x="3.91" y="3.9" radius="1.5" width="0.1524" layer="20"/>
-<circle x="3.91" y="72.29" radius="1.5" width="0.1524" layer="20"/>
-<circle x="69.877" y="72.29" radius="1.5" width="0.1524" layer="20"/>
-<circle x="69.877" y="3.9" radius="1.5" width="0.1524" layer="20"/>
-<circle x="65.897" y="7.632" radius="1.1305" width="0.1524" layer="20"/>
-<circle x="7.897" y="68.587" radius="1.1305" width="0.1524" layer="20"/>
-<circle x="65.877" y="68.587" radius="1.1305" width="0.1524" layer="20"/>
-<circle x="7.897" y="45.587" radius="1.1305" width="0.1524" layer="20"/>
-<circle x="65.877" y="45.587" radius="1.1305" width="0.1524" layer="20"/>
-<wire x1="7.874" y1="72.136" x2="8.001" y2="72.136" width="0.1524" layer="21"/>
-<wire x1="8.001" y1="72.136" x2="65.786" y2="72.136" width="0.1524" layer="21"/>
-<wire x1="65.786" y1="72.136" x2="69.342" y2="68.58" width="0.1524" layer="21" curve="-90"/>
-<wire x1="69.342" y1="68.58" x2="69.342" y2="45.466" width="0.1524" layer="21"/>
-<wire x1="69.342" y1="45.466" x2="65.913" y2="42.037" width="0.1524" layer="21" curve="-90"/>
-<wire x1="65.913" y1="42.037" x2="8.001" y2="42.037" width="0.1524" layer="21" locked="yes"/>
-<wire x1="8.001" y1="42.164" x2="4.572" y2="45.593" width="0.1524" layer="21" curve="-90"/>
-<wire x1="4.572" y1="45.593" x2="4.445" y2="45.72" width="0.1524" layer="21" curve="-90"/>
-<wire x1="4.445" y1="45.72" x2="4.445" y2="68.58" width="0.1524" layer="21"/>
-<wire x1="4.445" y1="68.58" x2="4.445" y2="69.088" width="0.1524" layer="21"/>
-<wire x1="4.445" y1="68.58" x2="8.001" y2="72.136" width="0.1524" layer="21" curve="-90"/>
-<circle x="7.987" y="30.614" radius="1.1305" width="0.1524" layer="20"/>
-<circle x="65.877" y="30.614" radius="1.1305" width="0.1524" layer="20"/>
-<circle x="7.897" y="7.614" radius="1.1305" width="0.1524" layer="20"/>
-<circle x="65.877" y="7.614" radius="1.1305" width="0.1524" layer="20"/>
-<wire x1="7.874" y1="34.163" x2="8.001" y2="34.163" width="0.1524" layer="21"/>
-<wire x1="8.001" y1="34.163" x2="65.786" y2="34.163" width="0.1524" layer="21" locked="yes"/>
-<wire x1="65.786" y1="34.163" x2="69.342" y2="30.607" width="0.1524" layer="21" curve="-90"/>
-<wire x1="69.342" y1="30.607" x2="69.342" y2="7.493" width="0.1524" layer="21"/>
-<wire x1="69.342" y1="7.493" x2="65.913" y2="4.064" width="0.1524" layer="21" curve="-90"/>
-<wire x1="65.913" y1="4.064" x2="8.001" y2="4.064" width="0.1524" layer="21"/>
-<wire x1="8.001" y1="4.191" x2="4.572" y2="7.62" width="0.1524" layer="21" curve="-90"/>
-<wire x1="4.572" y1="7.62" x2="4.445" y2="7.747" width="0.1524" layer="21" curve="-90"/>
-<wire x1="4.445" y1="7.747" x2="4.445" y2="30.607" width="0.1524" layer="21"/>
-<wire x1="4.445" y1="30.607" x2="4.445" y2="31.115" width="0.1524" layer="21"/>
-<wire x1="4.445" y1="30.607" x2="8.001" y2="34.163" width="0.1524" layer="21" curve="-90"/>
+<wire x1="1" y1="12" x2="0" y2="11" width="0.1524" layer="20" curve="90"/>
+<wire x1="0" y1="11" x2="0" y2="1" width="0.1524" layer="20"/>
+<wire x1="0" y1="1" x2="1" y2="0" width="0.1524" layer="20" curve="90"/>
+<wire x1="1" y1="0" x2="5" y2="0" width="0.1524" layer="20"/>
+<wire x1="7" y1="0" x2="11" y2="0" width="0.1524" layer="20"/>
+<wire x1="11" y1="0" x2="12" y2="1" width="0.1524" layer="20" curve="90"/>
+<wire x1="12" y1="1" x2="12" y2="11" width="0.1524" layer="20"/>
+<wire x1="12" y1="11" x2="11" y2="12" width="0.1524" layer="20" curve="90"/>
+<wire x1="11" y1="12" x2="1" y2="12" width="0.1524" layer="20"/>
+<rectangle x1="4.885" y1="1" x2="7.115" y2="11" layer="1"/>
+<rectangle x1="1" y1="1" x2="4" y2="11" layer="1"/>
+<polygon width="0.1016" layer="29" spacing="3.81">
+<vertex x="1" y="3"/>
+<vertex x="1" y="1"/>
+<vertex x="4" y="1"/>
+<vertex x="4" y="3"/>
+</polygon>
+<polygon width="0.1016" layer="30" spacing="3.81">
+<vertex x="1" y="3"/>
+<vertex x="1" y="1"/>
+<vertex x="4" y="1"/>
+<vertex x="4" y="3"/>
+</polygon>
+<polygon width="0.1016" layer="30" spacing="3.81">
+<vertex x="8" y="3"/>
+<vertex x="8" y="1"/>
+<vertex x="11" y="1"/>
+<vertex x="11" y="3"/>
+</polygon>
+<polygon width="0.1016" layer="29" spacing="3.81">
+<vertex x="8" y="3"/>
+<vertex x="8" y="1"/>
+<vertex x="11" y="1"/>
+<vertex x="11" y="3"/>
+</polygon>
+<wire x1="5" y1="0" x2="5" y2="3" width="0.1016" layer="20"/>
+<wire x1="5" y1="3" x2="7" y2="3" width="0.1016" layer="20"/>
+<wire x1="7" y1="3" x2="7" y2="0" width="0.1016" layer="20"/>
+<polygon width="0.1016" layer="34" spacing="3.81">
+<vertex x="4" y="3"/>
+<vertex x="4" y="4"/>
+<vertex x="8" y="4"/>
+<vertex x="8" y="3"/>
+</polygon>
+<polygon width="0.1016" layer="34" spacing="3.81">
+<vertex x="4" y="1"/>
+<vertex x="5" y="1"/>
+<vertex x="5" y="3"/>
+<vertex x="4" y="3"/>
+</polygon>
+<polygon width="0.1016" layer="30" spacing="3.81">
+<vertex x="7" y="4"/>
+<vertex x="7" y="1"/>
+<vertex x="8" y="1"/>
+<vertex x="8" y="4"/>
+</polygon>
+<polygon width="0.1016" layer="29" spacing="3.81">
+<vertex x="5" y="3"/>
+<vertex x="5" y="4"/>
+<vertex x="7" y="4"/>
+<vertex x="7" y="3"/>
+</polygon>
+<polygon width="0.1016" layer="29" spacing="3.81">
+<vertex x="5" y="11"/>
+<vertex x="5" y="10"/>
+<vertex x="7" y="10"/>
+<vertex x="7" y="11"/>
+</polygon>
 </plain>
 <attributes>
@@
 </elements>
 <signals>
+<signal name="GROUND">
+<polygon width="0.15" layer="16">
+<vertex x="-1" y="13"/>
+<vertex x="-1" y="-1"/>
+<vertex x="13" y="-1"/>
+<vertex x="13" y="13"/>
+</polygon>
+</signal>
+<signal name="S$1">
+<polygon width="0.15" layer="1">
+<vertex x="8" y="11"/>
+<vertex x="8" y="1"/>
+<vertex x="11" y="1"/>
+<vertex x="11" y="11"/>
+</polygon>
+</signal>
+<signal name="S$2">
+<via x="10" y="10" extent="1-16" drill="1" diameter="0.55"/>
+</signal>
+<signal name="S$3">
+<via x="2" y="10" extent="1-16" drill="1" diameter="0.55"/>
+</signal>
+<signal name="S$4">
+<via x="2" y="4" extent="1-16" drill="1" diameter="0.55"/>
+</signal>
+<signal name="S$5">
+<via x="10" y="4" extent="1-16" drill="1" diameter="0.55"/>
+</signal>
 </signals>
 </board>
 </drawing>
-<compatibility>
-<note version="8.5" severity="warning">
-Since Version 8.5, EAGLE supports locking for holes, vias, wires and polygons.
-The locking property on all objects of these types will not be understood in this version.
-</note>
-</compatibility>
 </eagle>
